File: Mid Board/HADES_motor_board/HADES_motor_board.kicad_pcb (KiCad board)
At the start: 2 copper layers, 142.8 x 139.9 mm, 0 parts

Commit message: v2
Routing:
- removed copper zone on B.Cu, net (none)
Other:
- board size 142.8 x 139.9 mm -> 145.8 x 136.7 mm
